File: minimal_adin1110/minimal_adin1110.kicad_sch (KiCad schematic)
At the start: 73 parts, among them J1 CLP-114-02-G-D-BE, J2 CLP-102-02-G-D-BE, J3 CLP-102-02-G-D-BE, J4 CLP-102-02-G-D-BE, J5 CLP-103-02-G-D-BE, U1 ADIN1110CCPZ, Y1 25.0000MHz

Commit message: Switch to KiCad 9
Changed lines of the file:
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@@
 (kicad_sch
-	(version 20231120)
+	(version 20250114)
 	(generator "eeschema")
-	(generator_version "8.0")
+	(generator_version "9.0")
 	(paper "A3")
 	(junction
@@
 		)
 	)
+	(embedded_fonts no)
 )

Commit message: development backup
Parts:
- removed J5: CLP-103-02-G-D-BE, connector_footprints:CLP-103-02-G-D-BE, symbol UNITED_CONNECTORS_DATA_BASE:J_CLP-103-02-G-D-BE
- removed MB5: mouse-bite-midle-50mil-200mil, mouse_bite_footprints:mouse-bite-midle-50mil-250mil, symbol UNITED_MOUSE_BITES_DATA_BASE:mouse-bite-midle-50mil-250mil
- removed TP22, TP23: TestPoint, test_point_footprints:TestPoint_THTPad_Castelated, symbol UNITED_TEST_POINTS:TestPoint_Castelated
- added C14, C5: 100 pF, capacitor_footprints:C_1812_4532Metric, symbol UNITED_CAPACITORS_DATA_BASE:C_C1812C101JHGACTU
- added D2: 3.3 V, diode_footprints:SOD323, symbol UNITED_DIODES_DATA_BASE:D_SP4020-01FTG-C
- added D4: 58 V, diode_footprints:DO-214AA, symbol UNITED_DIODES_DATA_BASE:D_SMBJ58CA
- added J4, J7: CLP-102-02-G-D-BE, connector_footprints:CLP-102-02-G-D-BE, symbol UNITED_CONNECTORS_DATA_BASE:J_CLP-102-02-G-D-BE
- added J6: TBP02R2-381, connector_footprints:TBP02R2-381-03BE, symbol UNITED_CONNECTORS_DATA_BASE:J_TBP02R2-381-03BE
- added L1: 470 µH, coupled_inductor_footprints:SRF0905A, symbol UNITED_COUPLED_INDUCTORS_DATA_BASE:L_SRF0905A-471Y
- added MB4, MB6: mouse-bite-midle-50mil-200mil, mouse_bite_footprints:mouse-bite-midle-50mil-200mil, symbol UNITED_MOUSE_BITES_DATA_BASE:mouse-bite-midle-50mil-200mil
- added R11, R2: 10 kΩ, resistor_footprints:R_0603_1608Metric, symbol UNITED_RESISTORS_DATA_BASE:R_ERJ-3EKF1002V
- added R15: 4.7 MΩ, resistor_footprints:R_2010_5025Metric, symbol UNITED_RESISTORS_DATA_BASE:R_CHV2010-JW-475ELF
- added TP10, TP11, TP20: TestPoint, test_point_footprints:TestPoint_THTPad_Castelated, symbol UNITED_TEST_POINTS:TestPoint_Castelated
- renumbered C3 to C1, C13 to C10, C1 to C11, C2 to C12, C14 to C13, C10 to C15, C8 to C16, C4 to C2, C5 to C3, C7 to C4, C11 to C7, C9 to C8, C12 to C9, D3 to D1, D4 to D3, D1 to D5, D2 to D6, J2 to J1, J3 to J2, J4 to J3, J1 to J5, MB2 to MB1, MB3 to MB2, MB4 to MB3, MB1 to MB5, R2 to R1, R12 to R10, R3 to R12, R4 to R13, R1 to R14, R11 to R3, R7 to R4, R8 to R5, R5 to R6, R6 to R7, R9 to R8, R10 to R9, TP15 to TP1, TP4 to TP12, TP5 to TP13, TP6 to TP14, TP7 to TP15, TP8 to TP16, TP9 to TP17, TP10 to TP18, TP11 to TP19, TP16 to TP2, TP12 to TP22, TP13 to TP23, TP14 to TP24, TP17 to TP3, TP18 to TP4, TP19 to TP5, TP20 to TP6, TP1 to TP7, TP2 to TP8, TP3 to TP9
Connections:
- net DATA_AND_POWER_N: now also TP21.1, J7.1, J7.3, L1.4, R11.2
- net DATA_AND_POWER_P: now also J4.2, J4.4, L1.2, R2.2, TP11.1; no longer TP21.1
- net GND: now also J4.1, J4.3, J7.2, J7.4, R15.2, TP10.1, TP20.1
- new net: D2.2, D4.1
- new net CABLE+: C5.1, D2.1, J6.1, L1.3, R2.1
- new net CABLE-: C14.1, D4.2, J6.2, L1.1, R11.1
- new net Earth: C14.2, C5.2, J6.3, R15.1
Other:
- moved on the sheet: C1, C10, C11, C12, C13, C15, C16, C2, C3, C4, C6, C7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

Commit message: development backup
Parts:
- removed C14, C5: 100 pF, capacitor_footprints:C_1812_4532Metric, symbol UNITED_CAPACITORS_DATA_BASE:C_C1812C101JHGACTU
- removed D2: 3.3 V, diode_footprints:SOD323, symbol UNITED_DIODES_DATA_BASE:D_SP4020-01FTG-C
- removed D4: 58 V, diode_footprints:DO-214AA, symbol UNITED_DIODES_DATA_BASE:D_SMBJ58CA
- removed J6: TBP02R2-381, connector_footprints:TBP02R2-381-03BE, symbol UNITED_CONNECTORS_DATA_BASE:J_TBP02R2-381-03BE
- removed L1: 470 µH, coupled_inductor_footprints:SRF0905A, symbol UNITED_COUPLED_INDUCTORS_DATA_BASE:L_SRF0905A-471Y
- removed R11, R2: 10 kΩ, resistor_footprints:R_0603_1608Metric, symbol UNITED_RESISTORS_DATA_BASE:R_ERJ-3EKF1002V
- removed R15: 4.7 MΩ, resistor_footprints:R_2010_5025Metric, symbol UNITED_RESISTORS_DATA_BASE:R_CHV2010-JW-475ELF
- renumbered C11 to C1, C15 to C10, C7 to C11, C9 to C12, C10 to C13, C13 to C14, C12 to C2, C1 to C3, C2 to C4, C3 to C5, C16 to C7, C4 to C8, C8 to C9, D5 to D1, D6 to D2, D1 to D3, D3 to D4, J5 to J1, J1 to J2, J2 to J3, J3 to J4, J4 to J5, J7 to J6, MB5 to MB1, MB1 to MB2, MB2 to MB3, MB3 to MB4, MB4 to MB5, R14 to R1, R9 to R10, R3 to R11, R10 to R12, R1 to R2, R12 to R3, R13 to R4, R6 to R5, R7 to R6, R4 to R7, R5 to R8, R8 to R9, TP7 to TP1, TP18 to TP10, TP19 to TP11, TP22 to TP12, TP23 to TP13, TP24 to TP14, TP1 to TP15, TP2 to TP16, TP3 to TP17, TP4 to TP18, TP5 to TP19, TP8 to TP2, TP6 to TP20, TP10 to TP21, TP11 to TP22, TP21 to TP23, TP20 to TP24, TP9 to TP3, TP12 to TP4, TP13 to TP5, TP14 to TP6, TP15 to TP7, TP16 to TP8, TP17 to TP9
Connections:
- net DATA_AND_POWER_N: now also J6.2, J6.4; no longer J6.1, J6.3
- net DATA_AND_POWER_P: now also J5.1, J5.3; no longer J5.2, J5.4
- net GND: now also J5.2, J5.4, J6.1, J6.3; no longer J5.1, J5.3, J6.2, J6.4
Other:
- moved on the sheet: C1, C10, C11, C12, C13, C14, C2, C3, C4, C5, C6, C7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

Commit message: development backup
Connections:
- net GND: now also J1.16; no longer J1.18
- net SPI_CFG1: now also J1.18; no longer J1.14
- net VDDIO: now also J1.14; no longer J1.16
Changed lines of the file:
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@@
-	(wire
-		(pts
-			(xy 125.73 153.67) (xy 128.27 153.67)
-		)
-		(stroke
-			(width 0)
-			(type default)
-		)
-	)
 	(wire
 		(pts
@@
 	(wire
 		(pts
-			(xy 125.73 151.13) (xy 130.81 151.13)
+			(xy 125.73 148.59) (xy 130.81 148.59)
 		)
 		(stroke
@@
 	(wire
 		(pts
+			(xy 128.27 151.13) (xy 125.73 151.13)
+		)
+		(stroke
+			(width 0)
+			(type default)
+		)
+	)
+	(wire
+		(pts
 			(xy 113.03 133.35) (xy 113.03 135.89)
 		)
@@
 	(wire
 		(pts
-			(xy 125.73 148.59) (xy 130.81 148.59)
+			(xy 125.73 153.67) (xy 130.81 153.67)
 		)
 		(stroke
@@
 	(wire
 		(pts
-			(xy 128.27 153.67) (xy 128.27 168.91)
+			(xy 128.27 151.13) (xy 128.27 168.91)
 		)
 		(stroke
@@
 	)
 	(label "SPI_CFG1"
-		(at 130.81 148.59 0)
+		(at 130.81 153.67 0)
 		(effects
 			(font
@@
 	)
 	(label "VDDIO"
-		(at 130.81 151.13 0)
+		(at 130.81 148.59 0)
 		(effects
 			(font
