File: minimal_adin1110/minimal_adin1110.kicad_pcb (KiCad board)
At the start: 4 copper layers, 46.4 x 27.9 mm, 71 parts, among them J1 CLP-114-02-G-D-BE, J2 CLP-102-02-G-D-BE, J3 CLP-102-02-G-D-BE, J4 CLP-102-02-G-D-BE, J5 CLP-103-02-G-D-BE, U1 ADIN1110CCPZ, Y1 25.0000MHz

Commit message: Update subproject commit for KiCAD Symbol Generator
Parts:
- added D3: 3.3 V, diode_footprints:SOD323, F.Cu at (149.2, 87.7)
- added D4: 3.3 V, diode_footprints:SOD323, F.Cu at (149.2, 91.3)
- moved J5 2.54 mm to (157.5, 88.9)
- moved MB5 2.54 mm to (154.1, 88.9)
- moved TP21 2.54 mm to (153.7, 88.9)
- moved TP22 2.54 mm to (153.7, 90.1)
- moved TP23 2.54 mm to (153.7, 87.6)
Routing:
- net /DATA_AND_POWER_P: track 4.19 -> 6.73 mm
- net /DATA_AND_POWER_N: track 4.19 -> 6.73 mm
- net GND: vias 115 -> 119
Other:
- board size 46.4 x 27.9 mm -> 48.9 x 27.9 mm

Commit message: Update minimal_adin1110 GLB file
Parts:
- moved FID3 19.1 mm to (150.2, 77.6)
- moved J5 5.23 mm to (157.5, 94.1)
- moved MB5 5.23 mm to (154.1, 94.1)
- moved TP21 5.23 mm to (153.7, 94.1)
- moved TP22 5.23 mm to (153.7, 95.4)
- moved TP23 5.23 mm to (153.7, 92.8)
Routing:
- net /DATA_AND_POWER_P: track 6.73 -> 9.99 mm
- net /DATA_AND_POWER_N: track 6.73 -> 9.99 mm
Other:
- outline, holes or cut-outs redrawn

Commit message: development backup
Parts:
- moved FID1 1.55 mm to (122.7, 77.3)
- moved FID2 1.55 mm to (122.7, 96.9)
- moved J1 1.27 mm to (117.2, 87.1)
- moved MB1 1.27 mm to (121.2, 87.1)
- moved TP1 1.27 mm to (121.7, 78.9)
- moved TP10 1.27 mm to (121.7, 90.3)
- moved TP11 1.27 mm to (121.7, 91.6)
- moved TP12 1.27 mm to (121.7, 92.8)
- moved TP13 1.27 mm to (121.7, 94.1)
- moved TP14 1.27 mm to (121.7, 95.4)
- moved TP2 1.27 mm to (121.7, 80.1)
- moved TP3 1.27 mm to (121.7, 81.4)
- moved TP4 1.27 mm to (121.7, 82.7)
- moved TP5 1.27 mm to (121.7, 83.9)
- moved TP6 1.27 mm to (121.7, 85.2)
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Routing:
- net /SCK: track 9.99 -> 8.70 mm
- net /TS_CAPT: track 10.2 -> 8.89 mm
- net /SPI_CFG1: track 9.89 -> 8.60 mm
- net /~{TX2P4_EN}: track 10.5 -> 9.18 mm
- net /~{SWPD_EN}: track 10.2 -> 8.91 mm
- net /~{CS}: track 12.6 -> 11.3 mm
- net /TS_TIMER__MS_SEL: track 11.3 -> 10.1 mm
- net /MOSI: track 11.1 -> 9.80 mm
- net /MISO: track 12.4 -> 11.1 mm
- net /LINK_ST: track 14.1 -> 12.8 mm
- net /~{RESET}: track 16.2 -> 14.9 mm
- net /~{INT}: track 14.9 -> 13.7 mm
- net GND: vias 119 -> 102
Other:
- board size 48.9 x 27.9 mm -> 47.6 x 27.9 mm

Commit message: Revert "development backup"
This reverts commit 9283c747e1c3676efe85313f236ce4507e137f4e.
Parts:
- moved FID1 1.55 mm to (124.2, 77.6)
- moved FID2 1.55 mm to (124.2, 96.6)
- moved J1 1.27 mm to (116.0, 87.1)
- moved MB1 1.27 mm to (119.9, 87.1)
- moved TP1 1.27 mm to (120.4, 78.9)
- moved TP10 1.27 mm to (120.4, 90.3)
- moved TP11 1.27 mm to (120.4, 91.6)
- moved TP12 1.27 mm to (120.4, 92.8)
- moved TP13 1.27 mm to (120.4, 94.1)
- moved TP14 1.27 mm to (120.4, 95.4)
- moved TP2 1.27 mm to (120.4, 80.1)
- moved TP3 1.27 mm to (120.4, 81.4)
- moved TP4 1.27 mm to (120.4, 82.7)
- moved TP5 1.27 mm to (120.4, 83.9)
- moved TP6 1.27 mm to (120.4, 85.2)
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Routing:
- net /SCK: track 8.70 -> 9.99 mm
- net /TS_CAPT: track 8.89 -> 10.2 mm
- net /SPI_CFG1: track 8.60 -> 9.89 mm
- net /~{TX2P4_EN}: track 9.18 -> 10.5 mm
- net /~{SWPD_EN}: track 8.91 -> 10.2 mm
- net /~{CS}: track 11.3 -> 12.6 mm
- net /TS_TIMER__MS_SEL: track 10.1 -> 11.3 mm
- net /MOSI: track 9.80 -> 11.1 mm
- net /MISO: track 11.1 -> 12.4 mm
- net /LINK_ST: track 12.8 -> 14.1 mm
- net /~{RESET}: track 14.9 -> 16.2 mm
- net /~{INT}: track 13.7 -> 14.9 mm
- net GND: vias 102 -> 119
Other:
- board size 47.6 x 27.9 mm -> 48.9 x 27.9 mm

Commit message: development backup
Parts:
- removed the J5 at (157.5, 94.1)
- removed the MB5 at (154.1, 94.1)
- removed the TP22 at (153.7, 95.4)
- removed the TP23 at (153.7, 92.8)
- added C14: 100 pF, capacitor_footprints:C_1812_4532Metric, F.Cu at (175.6, 89.2)
- added C5: 100 pF, capacitor_footprints:C_1812_4532Metric, F.Cu at (175.6, 81.3)
- added D2: 3.3 V, diode_footprints:SOD323, F.Cu at (163.4, 87.1)
- added D4: 58 V, diode_footprints:DO-214AA, F.Cu at (163.4, 92.8)
- added J4: CLP-102-02-G-D-BE, connector_footprints:CLP-102-02-G-D-BE, F.Cu at (154.4, 78.4)
- added J6: TBP02R2-381, connector_footprints:TBP02R2-381-03BE, F.Cu at (169.0, 87.1)
- added J7: CLP-102-02-G-D-BE, connector_footprints:CLP-102-02-G-D-BE, F.Cu at (154.4, 95.9)
- added L1: 470 µH, coupled_inductor_footprints:SRF0905A, F.Cu at (156.2, 87.1)
- added MB4: mouse-bite-midle-50mil-200mil, mouse_bite_footprints:mouse-bite-midle-50mil-200mil, F.Cu at (154.4, 80.9)
- added MB6: mouse-bite-midle-50mil-200mil, mouse_bite_footprints:mouse-bite-midle-50mil-200mil, F.Cu at (154.4, 93.3)
- added R11: 10 kΩ, resistor_footprints:R_0603_1608Metric, F.Cu at (157.2, 91.3)
- added R15: 4.7 MΩ, resistor_footprints:R_2010_5025Metric, F.Cu at (170.2, 95.3)
- added R2: 10 kΩ, resistor_footprints:R_0603_1608Metric, F.Cu at (157.2, 83.0)
- added TP10: TestPoint, test_point_footprints:TestPoint_THTPad_Castelated, F.Cu at (153.8, 81.5)
- added TP11: TestPoint, test_point_footprints:TestPoint_THTPad_Castelated, F.Cu at (155.1, 81.5)
- added TP20: TestPoint, test_point_footprints:TestPoint_THTPad_Castelated, F.Cu at (153.8, 92.7)
- moved FID3 34.2 mm to (178.4, 96.9)
- moved D1 5.34 mm to (148.9, 82.4), turned to 180 degrees
- moved C10 3.65 mm to (149.2, 86.0)
- moved C13 3.65 mm to (149.2, 88.2)
- moved R10 3.65 mm to (149.2, 90.1)
- moved R3 3.65 mm to (149.2, 84.1)
- moved R4 3.65 mm to (145.9, 84.6)
- moved R5 3.65 mm to (145.9, 86.3)
- moved R7 3.65 mm to (143.4, 87.4)
- moved R8 3.65 mm to (145.9, 88.0)
- moved R9 3.65 mm to (145.9, 89.6)
- moved R6 3.65 mm to (141.7, 86.6)
- moved TP21 1.97 mm to (155.1, 92.7), turned to 90 degrees
- moved FID1 1.55 mm to (122.7, 77.3)
- moved FID2 1.55 mm to (122.7, 96.9)
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- renumbered C3 to C1, C13 to C10, C1 to C11, C2 to C12, C14 to C13, C10 to C15, C8 to C16, C4 to C2, C5 to C3, C7 to C4, C11 to C7, C9 to C8, C12 to C9, D3 to D1, D4 to D3, D1 to D5, D2 to D6, J2 to J1, J3 to J2, J4 to J3, J1 to J5, MB2 to MB1, MB3 to MB2, MB4 to MB3, MB1 to MB5, R2 to R1, R12 to R10, R3 to R12, R4 to R13, R1 to R14, R11 to R3, R7 to R4, R8 to R5, R5 to R6, R6 to R7, R9 to R8, R10 to R9, TP15 to TP1, TP4 to TP12, TP5 to TP13, TP6 to TP14, TP7 to TP15, TP8 to TP16, TP9 to TP17, TP10 to TP18, TP11 to TP19, TP16 to TP2, TP12 to TP22, TP13 to TP23, TP14 to TP24, TP17 to TP3, TP18 to TP4, TP19 to TP5, TP20 to TP6, TP1 to TP7, TP2 to TP8, TP3 to TP9
Connections:
- TP21 pad 1: /DATA_AND_POWER_P -> /DATA_AND_POWER_N
Routing:
- net /DATA_AND_POWER_N: track 9.99 -> 0.00 mm
- net /DATA_AND_POWER_P: track 9.99 -> 0.00 mm
- net /TXP: track 7.95 -> 11.0 mm
- net /RXP: track 7.82 -> 10.7 mm
- net /RXN: track 8.01 -> 10.6 mm
- net /TXN: track 8.58 -> 11.0 mm
- net Net-(D2-Pad2): track 0.00 -> 2.04 mm
- net /SCK: track 9.99 -> 8.70 mm
- net /~{TX2P4_EN}: track 10.5 -> 9.18 mm
- net /~{SWPD_EN}: track 10.2 -> 8.91 mm
- net /~{CS}: track 12.6 -> 11.3 mm
- net /TS_TIMER__MS_SEL: track 11.3 -> 10.1 mm
- net /MOSI: track 11.1 -> 9.80 mm
- net /MISO: track 12.4 -> 11.1 mm
- net /LINK_ST: track 14.1 -> 12.8 mm
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- added copper zone on F.Cu, net /CABLE+
- added copper zone on F.Cu, net /CABLE-
- added copper zone on F.Cu, net Earth
- added copper zone on In1.Cu, net Earth
Other:
- board size 48.9 x 27.9 mm -> 66 x 27.9 mm
