File: minimal_adin1110/minimal_adin1110.kicad_pcb (KiCad board)
At the start: 4 copper layers, 66 x 27.9 mm, 85 parts, among them J1 CLP-102-02-G-D-BE, J2 CLP-102-02-G-D-BE, J3 CLP-102-02-G-D-BE, J4 CLP-102-02-G-D-BE, J5 CLP-114-02-G-D-BE, J6 TBP02R2-381, J7 CLP-102-02-G-D-BE, U1 ADIN1110CCPZ, Y1 25.0000MHz

Commit message: development backup
Other:
- board size 66 x 27.9 mm -> 66 x 27.7 mm

Commit message: development backup
Parts:
- removed the C14 at (175.6, 89.2)
- removed the C5 at (175.6, 81.3)
- removed the D2 at (163.4, 87.1)
- removed the D4 at (163.4, 92.8)
- removed the J6 at (169.0, 87.1)
- removed L1: 470 µH, coupled_inductor_footprints:SRF0905A
- removed the R11 at (157.2, 91.3)
- removed R15: 4.7 MΩ, resistor_footprints:R_2010_5025Metric
- removed the R2 at (157.2, 83.0)
- moved FID3 40.0 mm to (138.4, 96.9)
- moved J5 6.19 mm to (157.1, 83.9), turned to 180 degrees
- moved J6 6.19 mm to (157.1, 90.3), turned to 180 degrees
- moved TP22 3.30 mm to (153.8, 84.6), turned to 180 degrees
- moved TP23 3.30 mm to (153.8, 89.7), turned to 180 degrees
- moved MB5 3.05 mm to (154.4, 83.9), turned to -90 degrees
- moved MB6 3.05 mm to (154.4, 90.3), turned to -90 degrees
- moved TP21 1.78 mm to (153.8, 83.3), turned to 180 degrees
- moved TP24 1.78 mm to (153.8, 90.9), turned to 180 degrees
- renumbered C11 to C1, C15 to C10, C7 to C11, C9 to C12, C10 to C13, C13 to C14, C12 to C2, C1 to C3, C2 to C4, C3 to C5, C16 to C7, C4 to C8, C8 to C9, D5 to D1, D6 to D2, D1 to D3, D3 to D4, J5 to J1, J1 to J2, J2 to J3, J3 to J4, J4 to J5, J7 to J6, MB5 to MB1, MB1 to MB2, MB2 to MB3, MB3 to MB4, MB4 to MB5, R14 to R1, R9 to R10, R3 to R11, R10 to R12, R1 to R2, R12 to R3, R13 to R4, R6 to R5, R7 to R6, R4 to R7, R5 to R8, R8 to R9, TP7 to TP1, TP18 to TP10, TP19 to TP11, TP22 to TP12, TP23 to TP13, TP24 to TP14, TP1 to TP15, TP2 to TP16, TP3 to TP17, TP4 to TP18, TP5 to TP19, TP8 to TP2, TP6 to TP20, TP10 to TP21, TP11 to TP22, TP21 to TP23, TP20 to TP24, TP9 to TP3, TP12 to TP4, TP13 to TP5, TP14 to TP6, TP15 to TP7, TP16 to TP8, TP17 to TP9
Connections:
- J5 pad 1: GND -> /DATA_AND_POWER_P
- J5 pad 2: /DATA_AND_POWER_P -> GND
- J5 pad 3: GND -> /DATA_AND_POWER_P
- J5 pad 4: /DATA_AND_POWER_P -> GND
- J6 pad 1: /DATA_AND_POWER_N -> GND
- J6 pad 2: GND -> /DATA_AND_POWER_N
- J6 pad 3: /DATA_AND_POWER_N -> GND
- J6 pad 4: GND -> /DATA_AND_POWER_N
Routing:
- net Net-(D2-Pad2): track 2.04 -> 0.00 mm
- net GND: vias 89 -> 79
- net Earth: vias 8 -> 0
- removed copper zone on F.Cu, net /CABLE+
- removed copper zone on F.Cu, net /CABLE-
- removed copper zone on F.Cu, net Earth
- removed copper zone on In1.Cu, net Earth
Other:
- board size 66 x 27.7 mm -> 46.5 x 27.7 mm

Commit message: development backup
Parts:
- moved FID1 30.6 mm to (153.0, 81.0)
- moved FID2 30.6 mm to (153.0, 93.2)
- moved JP3 3.56 mm to (144.5, 81.0), turned to 0 degrees
- moved TP8 2.67 mm to (121.7, 85.1)
- moved JP2 2.23 mm to (141.2, 81.4)
- moved C2 1.30 mm to (126.8, 87.7)
- moved C1 1.28 mm to (125.3, 87.7)
- moved E1 1.27 mm to (138.1, 82.1)
- moved MB2 1.27 mm to (128.7, 77.0)
- moved MB3 1.27 mm to (136.9, 77.0)
- moved MB4 1.27 mm to (145.2, 77.0)
- moved Y1 1.27 mm to (136.6, 93.9)
- moved C10 1.27 mm to (136.8, 92.0)
- moved C3 1.27 mm to (132.3, 82.1)
- moved C4 1.27 mm to (133.4, 82.1)
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Connections:
- J1 pad 14: /SPI_CFG1 -> /VDDIO
- J1 pad 16: /VDDIO -> GND
- J1 pad 18: GND -> /SPI_CFG1
Routing:
- net /SPI_CFG1: track 8.62 -> 11.1 mm
- net /TXP: track 11.0 -> 12.3 mm
- net /~{RESET}: track 14.9 -> 13.9 mm
- net /RXP: track 10.7 -> 11.6 mm
- net /VDDIO: track 3.78 -> 3.02 mm
- net Net-(U1-LED_0): track 3.86 -> 3.22 mm
- net /RXN: track 10.6 -> 11.2 mm
- net /TS_TIMER__MS_SEL: track 10.1 -> 10.6 mm
- net Net-(U1-LED_1): track 4.25 -> 3.71 mm
- net /LINK_ST: track 12.8 -> 12.3 mm
- net /~{INT}: track 13.7 -> 14.2 mm
- net /~{CS}: track 11.3 -> 11.8 mm
- net GND: vias 79 -> 48
Other:
- board size 46.5 x 27.7 mm -> 46.5 x 26.2 mm
